File: KiCad/KiCad.kicad_pcb (KiCad board)
At the start: 2 copper layers, 72.5 x 40 mm, 18 parts, among them J1 Conn_02x03, SW1 SW_Push, SW2 SW_Push, SW3 SW_Push, U1 ATmega48A-P, Y1 Quartz Crystal

Commit message: Changes to PCB
Parts:
- moved J1 7.07 mm to (62.5, 60.0), turned to -90 degrees
- moved BT1 2.50 mm to (57.5, 40.0)
Routing:
- net Net-(J1-Pin_3): track 10.2 -> 29.0 mm
- net Net-(BT1-+): track 46.1 -> 53.0 mm
- net Net-(J1-Pin_6): track 50.7 -> 49.2 mm
- net Net-(J1-Pin_2): track 11.6 -> 12.6 mm
Changed lines of the file:
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@@
   )
   (footprint "Connector_PinSocket_2.54mm:PinSocket_2x03_P2.54mm_Vertical" (layer "F.Cu")
-    (at 67.5 54.960001)
+    (at 62.54 60 -90)
     (descr "Through hole straight socket strip, 2x03, 2.54mm pitch, double cols (from Kicad 4.0.7), script generated")
     (tags "Through hole socket strip THT 2x03 2.54mm double row")
@@
     (property "ki_keywords" "connector")
     (attr through_hole)
-    (fp_text reference "J1" (at -5 5.04 90) (layer "F.SilkS") hide
-        (effects (font (size 1 1) (thickness 0.15)))
-    )
-    (fp_text value "Conn_02x03" (at -1.27 7.85) (layer "F.Fab") hide
-        (effects (font (size 1 1) (thickness 0.15)))
-    )
-    (fp_text user "${REFERENCE}" (at -1.27 2.54 90) (layer "F.Fab")
+    (fp_text reference "J1" (at -5 5.04) (layer "F.SilkS") hide
+        (effects (font (size 1 1) (thickness 0.15)))
+    )
+    (fp_text value "Conn_02x03" (at -1.27 7.85 90) (layer "F.Fab") hide
+        (effects (font (size 1 1) (thickness 0.15)))
+    )
+    (fp_text user "${REFERENCE}" (at -1.27 2.54) (layer "F.Fab")
         (effects (font (size 1 1) (thickness 0.15)))
     )
@@
     (fp_line (start 1.27 6.35) (end -3.81 6.35)
       (stroke (width 0.1) (type solid)) (layer "F.Fab"))
-    (pad "1" thru_hole rect (at 0 0) (size 1.7 1.7) (drill 1) (layers "*.Cu" "*.Mask")
+    (pad "1" thru_hole rect (at 0 0 270) (size 1.7 1.7) (drill 1) (layers "*.Cu" "*.Mask")
       (net 1 "Net-(BT1-+)") (pinfunction "Pin_1") (pintype "passive"))
-    (pad "2" thru_hole oval (at -2.54 0) (size 1.7 1.7) (drill 1) (layers "*.Cu" "*.Mask")
+    (pad "2" thru_hole oval (at -2.54 0 270) (size 1.7 1.7) (drill 1) (layers "*.Cu" "*.Mask")
       (net 15 "Net-(J1-Pin_2)") (pinfunction "Pin_2") (pintype "passive"))
-    (pad "3" thru_hole oval (at 0 2.54) (size 1.7 1.7) (drill 1) (layers "*.Cu" "*.Mask")
+    (pad "3" thru_hole oval (at 0 2.54 270) (size 1.7 1.7) (drill 1) (layers "*.Cu" "*.Mask")
       (net 16 "Net-(J1-Pin_3)") (pinfunction "Pin_3") (pintype "passive"))
-    (pad "4" thru_hole oval (at -2.54 2.54) (size 1.7 1.7) (drill 1) (layers "*.Cu" "*.Mask")
+    (pad "4" thru_hole oval (at -2.54 2.54 270) (size 1.7 1.7) (drill 1) (layers "*.Cu" "*.Mask")
       (net 17 "Net-(J1-Pin_4)") (pinfunction "Pin_4") (pintype "passive"))
-    (pad "5" thru_hole oval (at 0 5.08) (size 1.7 1.7) (drill 1) (layers "*.Cu" "*.Mask")
+    (pad "5" thru_hole oval (at 0 5.08 270) (size 1.7 1.7) (drill 1) (layers "*.Cu" "*.Mask")
       (net 22 "GND") (pinfunction "Pin_5") (pintype "passive"))
-    (pad "6" thru_hole oval (at -2.54 5.08) (size 1.7 1.7) (drill 1) (layers "*.Cu" "*.Mask")
+    (pad "6" thru_hole oval (at -2.54 5.08 270) (size 1.7 1.7) (drill 1) (layers "*.Cu" "*.Mask")
       (net 18 "Net-(J1-Pin_6)") (pinfunction "Pin_6") (pintype "passive"))
     (model "${KICAD6_3DMODEL_DIR}/Connector_PinSocket_2.54mm.3dshapes/PinSocket_2x03_P2.54mm_Vertical.wrl"
@@
   )
   (footprint "Battery:BatteryHolder_Keystone_106_1x20mm" (layer "F.Cu")
-    (at 57.5 42.500001 180)
+    (at 57.5 40.000001 180)
     (descr "http://www.keyelco.com/product-pdf.cfm?p=720")
     (tags "Keystone type 106 battery holder")
@@
     (stroke (width 0.1) (type default)) (layer "Edge.Cuts"))
   (segment (start 82.26 45.240001) (end 82.26 42.380001) (width 0.8) (layer "B.Cu") (net 1))
-  (segment (start 67.5 54.960001) (end 67.5 54.600001) (width 0.8) (layer "B.Cu") (net 1))
+  (segment (start 57.5 40.000001) (end 65 47.500001) (width 0.8) (layer "B.Cu") (net 1))
   (segment (start 80 47.500001) (end 82.26 45.240001) (width 0.8) (layer "B.Cu") (net 1))
   (segment (start 77.5 47.500001) (end 77.18 47.820001) (width 0.8) (layer "B.Cu") (net 1))
   (segment (start 77.5 47.500001) (end 80 47.500001) (width 0.8) (layer "B.Cu") (net 1))
-  (segment (start 62.5 47.500001) (end 77.5 47.500001) (width 0.8) (layer "B.Cu") (net 1))
-  (segment (start 72.460001 54.960001) (end 67.5 54.960001) (width 0.8) (layer "B.Cu") (net 1))
-  (segment (start 73.311371 55) (end 72.5 55) (width 0.8) (layer "B.Cu") (net 1))
+  (segment (start 65 47.500001) (end 77.5 47.500001) (width 0.8) (layer "B.Cu") (net 1))
   (segment (start 77.18 47.820001) (end 77.18 50.000001) (width 0.8) (layer "B.Cu") (net 1))
-  (segment (start 77.18 51.131371) (end 73.311371 55) (width 0.8) (layer "B.Cu") (net 1))
-  (segment (start 62.5 47.500001) (end 57.5 42.500001) (width 0.8) (layer "B.Cu") (net 1))
-  (segment (start 77.18 50.000001) (end 77.18 51.131371) (width 0.8) (layer "B.Cu") (net 1))
-  (segment (start 72.5 55) (end 72.460001 54.960001) (width 0.8) (layer "B.Cu") (net 1))
+  (segment (start 62.58 60) (end 67.180001 60) (width 0.8) (layer "B.Cu") (net 1))
+  (segment (start 67.180001 60) (end 77.18 50.000001) (width 0.8) (layer "B.Cu") (net 1))
   (segment (start 75 27.500001) (end 85 37.500001) (width 0.8) (layer "B.Cu") (net 2))
   (segment (start 85 37.500001) (end 85 40.040001) (width 0.8) (layer "B.Cu") (net 2))
@@
   (segment (start 72.5 40.240001) (end 74.64 42.380001) (width 0.8) (layer "B.Cu") (net 14))
   (segment (start 72.5 37.500001) (end 72.5 40.240001) (width 0.8) (layer "B.Cu") (net 14))
-  (segment (start 65.21792 53.5) (end 64.96 53.75792) (width 0.8) (layer "B.Cu") (net 15))
-  (segment (start 64.96 53.75792) (end 64.96 54.960001) (width 0.8) (layer "B.Cu") (net 15))
-  (segment (start 71.5 53.5) (end 65.21792 53.5) (width 0.8) (layer "B.Cu") (net 15))
-  (segment (start 72.1 52.9) (end 72.1 50.000001) (width 0.8) (layer "B.Cu") (net 15))
-  (segment (start 71.5 53.5) (end 72.1 52.9) (width 0.8) (layer "B.Cu") (net 15))
-  (segment (start 70 57.5) (end 70 52.5) (width 0.8) (layer "F.Cu") (net 16))
-  (via (at 70 57.5) (size 0.8) (drill 0.4) (layers "F.Cu" "B.Cu") (net 16))
-  (via (at 70 52.5) (size 0.8) (drill 0.4) (layers "F.Cu" "B.Cu") (net 16))
-  (segment (start 70 52.5) (end 70 50.440001) (width 0.8) (layer "B.Cu") (net 16))
-  (segment (start 70 50.440001) (end 69.56 50.000001) (width 0.8) (layer "B.Cu") (net 16))
-  (segment (start 67.5 57.500001) (end 70 57.5) (width 0.8) (layer "B.Cu") (net 16))
-  (segment (start 73.975336 51.5) (end 66 51.5) (width 0.8) (layer "F.Cu") (net 17))
-  (segment (start 66 51.5) (end 65 52.5) (width 0.8) (layer "F.Cu") (net 17))
-  (segment (start 74.037418 51.562082) (end 73.975336 51.5) (width 0.8) (layer "F.Cu") (net 17))
-  (via (at 65 52.5) (size 0.8) (drill 0.4) (layers "F.Cu" "B.Cu") (net 17))
-  (via (at 74.037418 51.562082) (size 0.8) (drill 0.4) (layers "F.Cu" "B.Cu") (net 17))
-  (segment (start 74.64 51.562082) (end 74.037418 51.562082) (width 0.8) (layer "B.Cu") (net 17))
-  (segment (start 63.51 53.793706) (end 63.51 56.050001) (width 0.8) (layer "B.Cu") (net 17))
-  (segment (start 65 52.5) (end 64.803706 52.5) (width 0.8) (layer "B.Cu") (net 17))
-  (segment (start 64.803706 52.5) (end 63.51 53.793706) (width 0.8) (layer "B.Cu") (net 17))
-  (segment (start 63.51 56.050001) (end 64.96 57.500001) (width 0.8) (layer "B.Cu") (net 17))
-  (segment (start 74.64 51.562082) (end 74.64 50.000001) (width 0.8) (layer "B.Cu") (net 17))
+  (segment (start 64.640001 57.46) (end 72.1 50.000001) (width 0.8) (layer "B.Cu") (net 15))
+  (segment (start 62.58 57.46) (end 64.640001 57.46) (width 0.8) (layer "B.Cu") (net 15))
+  (segment (start 55.5 54.5) (end 55.5 61) (width 0.8) (layer "F.Cu") (net 16))
+  (segment (start 56.25 61.75) (end 60 61.75) (width 0.8) (layer "F.Cu") (net 16))
+  (segment (start 56.25 53.75) (end 55.5 54.5) (width 0.8) (layer "F.Cu") (net 16))
+  (segment (start 63.5 53.75) (end 56.25 53.75) (width 0.8) (layer "F.Cu") (net 16))
+  (segment (start 55.5 61) (end 56.25 61.75) (width 0.8) (layer "F.Cu") (net 16))
+  (via (at 60 61.75) (size 0.8) (drill 0.4) (layers "F.Cu" "B.Cu") (net 16))
+  (via (at 63.5 53.75) (size 0.8) (drill 0.4) (layers "F.Cu" "B.Cu") (net 16))
+  (segment (start 60 60) (end 60 61.75) (width 0.8) (layer "B.Cu") (net 16))
+  (segment (start 69.56 50.000001) (end 65.810001 53.75) (width 0.8) (layer "B.Cu") (net 16))
+  (segment (start 65.810001 53.75) (end 63.5 53.75) (width 0.8) (layer "B.Cu") (net 16))
+  (segment (start 65 55) (end 70 55) (width 0.8) (layer "F.Cu") (net 17))
+  (via (at 65 55) (size 0.8) (drill 0.4) (layers "F.Cu" "B.Cu") (net 17))
+  (via (at 70 55) (size 0.8) (drill 0.4) (layers "F.Cu" "B.Cu") (net 17))
+  (segment (start 70 55) (end 70 54.640001) (width 0.8) (layer "B.Cu") (net 17))
+  (segment (start 60.04 57.46) (end 62.5 55) (width 0.8) (layer "B.Cu") (net 17))
+  (segment (start 62.5 55) (end 65 55) (width 0.8) (layer "B.Cu") (net 17))
+  (segment (start 70 54.640001) (end 74.64 50.000001) (width 0.8) (layer "B.Cu") (net 17))
   (segment (start 62.5 47.5) (end 62.5 52.5) (width 0.8) (layer "F.Cu") (net 18))
   (segment (start 85 45) (end 65 45) (width 0.8) (layer "F.Cu") (net 18))
@@
   (via (at 85 45) (size 0.8) (drill 0.4) (layers "F.Cu" "B.Cu") (net 18))
   (via (at 62.5 52.5) (size 0.8) (drill 0.4) (layers "F.Cu" "B.Cu") (net 18))
+  (segment (start 62.42 52.5) (end 62.5 52.5) (width 0.25) (layer "B.Cu") (net 18))
   (segment (start 94.880001 45) (end 85 45) (width 0.8) (layer "B.Cu") (net 18))
   (segment (start 97.5 42.380001) (end 94.880001 45) (width 0.8) (layer "B.Cu") (net 18))
-  (segment (start 62.5 52.5) (end 62.5 57.580001) (width 0.8) (layer "B.Cu") (net 18))
-  (segment (start 62.5 57.580001) (end 64.96 60.040001) (width 0.8) (layer "B.Cu") (net 18))
+  (segment (start 57.46 57.46) (end 62.42 52.5) (width 0.8) (layer "B.Cu") (net 18))
   (segment (start 94.96 40.040001) (end 94.96 42.380001) (width 0.8) (layer "B.Cu") (net 19))
   (segment (start 97.5 35.000001) (end 97.5 37.500001) (width 0.8) (layer "B.Cu") (net 19))
